File: hardware/routine-quest.kicad_sch (KiCad schematic)
At the start: 90 parts, among them J1 USB4105-GF-A, J2 BTN1, J3 BTN2, J4 BTN3, J5 BTN4, Q1 2N7002, SW1 RESET, SW2 BOOT, U1 ESP32-S3-WROOM-1-N8, U2 USBLC6-2SC6, U3 TPS22918DBVR, U4 AP7361C-33E-13, U5 74AHCT1G125

Commit message: feat(hardware): PCB layout WIP — placement, autorouting pipeline, checks (phase 6b)
Work in progress, NOT for ordering (see docs/06b-pcb.md "Πού έμεινε").

- gen_pcb.py: main board 100x100 mm 2L (ESP32 antenna at edge + keep-out, USB-C left edge,
  12-LED ring, LDO/load switch inside ring, JSTs in corners, bottom test pads), button board
  24x24 mm; net classes, design rules, GND pours, stitching vias; parts/nets from gen_schematics
- route_pcb.py: Freerouting 1.9.0 via DSN/SES (own SES parser), zone fill, DRC report
- check_pcb.py: board nets == schematic, DRC, antenna clearance, USB-C at edge
- Footprints: new RQ:Buzzer_MLT-8530 (verify vs manufacturer drawing), vendored Espressif
  ESP32-S3-WROOM-1; project fp-lib-table; USB-C-only DRC rule
- Schematic: BZ1 footprint field set to RQ:Buzzer_MLT-8530 (no electrical change)
- Status: button board routed, DRC clean; main board 8 unconnected (USB-C fan-out, GND islands)

Co-Authored-By: Claude Opus 5.5 <noreply@anthropic.com>
Claude-Session: https://claude.ai/code/session_018m2P3s8baNXUUh6XjxJz11
Parts:
- BZ1: footprint RQ:Buzzer_MLT-8530 (create in Phase 6b) -> RQ:Buzzer_MLT-8530
Changed lines of the file:
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@@
     (property "Reference" "BZ1" (at 339.09 203.835 0) (effects (font (size 1.27 1.27))))
     (property "Value" "MLT-8530" (at 339.09 210.185 0) (effects (font (size 1.27 1.27))))
-    (property "Footprint" "RQ:Buzzer_MLT-8530 (create in Phase 6b)" (at 339.09 207.01 0) (effects (font (size 1.27 1.27)) hide))
+    (property "Footprint" "RQ:Buzzer_MLT-8530" (at 339.09 207.01 0) (effects (font (size 1.27 1.27)) hide))
     (property "Datasheet" "~" (at 339.09 207.01 0) (effects (font (size 1.27 1.27)) hide))
     (property "MPN" "MLT-8530" (at 339.09 207.01 0) (effects (font (size 1.27 1.27)) hide))
